File: UrchinCam_Expander_PCBA_01/UrchinCam_01.kicad_pcb (KiCad board)
At the start: 4 copper layers, 31.5 x 65 mm, 92 parts, among them J1 95157-440LF, J2 SM04B-GHS, J3 SM04B-GHS, J4 SM02B-GHS, J5 SM04B-GHS, U1 MP6550, U2 ADS1115IDGS, U3 BNO085, U4 TSR 3-2450N, U5 RTL8152B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

Commit message: Incorporated feedback from meeting.
Parts:
- removed the G*** at (151.6, 75.9)
- added FID1: Fiducial, Fiducial:Fiducial_0.5mm_Mask1mm, F.Cu at (137.0, 130.5)
- added FID2: Fiducial, Fiducial:Fiducial_0.5mm_Mask1mm, F.Cu at (163.9, 78.0)
- added FID3: Fiducial, Fiducial:Fiducial_0.5mm_Mask1mm, B.Cu at (137.0, 130.5)
- added FID4: Fiducial, Fiducial:Fiducial_0.5mm_Mask1mm, B.Cu at (163.9, 78.0)
- added J6: SM02B-GHS, Connector_JST:JST_GH_SM02B-GHS-TB_1x02-1MP_P1.25mm_Horizontal, B.Cu at (151.4, 76.5)
- moved C1 1.54 mm to (155.2, 82.6)
- moved C2 1.54 mm to (158.8, 84.8)
- moved C30 1.54 mm to (158.8, 83.5)
- moved C29 1.54 mm to (155.2, 84.4)
- moved U4 1.50 mm to (157.5, 87.2)
Routing:
- net Net-(J4-Pin_1): track 16.7 -> 14.9 mm
- net +5V: track 114.5 -> 115.2 mm, vias 9 -> 12
- net GND: vias 44 -> 48
Other:
- board text added: "+"
- board text added: "-"
- board text added: "5V (BATT EXT)"
