File: UrchinCam_Expander_PCBA_01/UrchinCam_01.kicad_sch (KiCad schematic)
At the start: 95 parts, among them J1 95157-440LF, J2 SM04B-GHS, J3 SM04B-GHS, J4 SM02B-GHS, J5 SM04B-GHS, J6 SM02B-GHS, U1 MP6550, U2 ADS1115IDGS, U3 BNO085, U4 TSR 3-2450N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

Commit message: Last edits!
Other:
- note added: "Jan 16, 2026"
- note added: "M2.5 Unplated Mounting Holes"
- note added: "Pi USB"
- note added: "Urchin Cam Expander PCBA"
- note added: "UrchinCam"
- note added: "v0.1"
- note removed: "M2.5 Unplated TH Mounting"
- note removed: "TH Header to Pi USB"
- moved on the sheet: H1, H2, H3, H4
Changed lines of the file:
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@@
 		)
 	)
+	(text "UrchinCam"
+		(exclude_from_sim no)
+		(at 352.806 261.112 0)
+		(effects
+			(font
+				(size 4.064 4.064)
+				(thickness 0.8128)
+				(bold yes)
+				(color 0 0 0 0.75)
+			)
+		)
+	)
+	(text "Urchin Cam Expander PCBA"
+		(exclude_from_sim no)
+		(at 333.248 276.86 0)
+		(effects
+			(font
+				(size 2.032 2.032)
+				(color 0 0 0 1)
+			)
+		)
+	)
 	(text "Power rail test points"
 		(exclude_from_sim no)
@@
 		)
 	)
-	(text "M2.5 Unplated TH Mounting"
+	(text "M2.5 Unplated Mounting Holes"
 		(exclude_from_sim no)
-		(at 341.63 147.828 0)
+		(at 341.63 142.748 0)
 		(effects
 			(font
@@
 		)
 	)
-	(text "TH Header\nto Pi USB"
+	(text "Pi USB"
 		(exclude_from_sim no)
 		(at 148.59 229.87 0)
@@
 		)
 	)
+	(text "v0.1"
+		(exclude_from_sim no)
+		(at 398.272 280.416 0)
+		(effects
+			(font
+				(size 2.032 2.032)
+				(color 0 0 0 1)
+			)
+		)
+	)
 	(text "IMU\n"
 		(exclude_from_sim no)
@@
 		)
 	)
+	(text "Jan 16, 2026"
+		(exclude_from_sim no)
+		(at 343.916 280.416 0)
+		(effects
+			(font
+				(size 2.032 2.032)
+				(color 0 0 0 1)
+			)
+		)
+	)
 	(text "ADDR: 0x48"
 		(exclude_from_sim no)
@@
 	(symbol
 		(lib_id "Mounting_Holes:Mounting_Hole_M2.5")
-		(at 320.04 140.97 0)
+		(at 320.04 135.89 0)
 		(unit 1)
 		(exclude_from_sim no)
@@
 		(fields_autoplaced yes)
 		(property "Reference" "H1"
-			(at 322.58 139.6999 0)
+			(at 322.58 134.6199 0)
 			(effects
 				(font
@@
 		)
 		(property "Value" "M2.5"
-			(at 322.58 142.2399 0)
+			(at 322.58 137.1599 0)
 			(effects
 				(font
@@
 		)
 		(property "Footprint" "Mounting_Holes:M2.5_Mounting_Hole_2.9mm_unplated"
-			(at 321.056 146.05 0)
+			(at 321.056 140.97 0)
 			(effects
 				(font
@@
 		)
 		(property "Datasheet" ""
-			(at 320.04 140.97 0)
+			(at 320.04 135.89 0)
 			(effects
 				(font
@@
 		)
 		(property "Description" "Mounting Hole M2.5 unplated 2.9mm diameter"
-			(at 320.294 148.336 0)
+			(at 320.294 143.256 0)
 			(effects
 				(font
@@
 	(symbol
 		(lib_id "Mounting_Holes:Mounting_Hole_M2.5")
-		(at 358.14 140.97 0)
+		(at 358.14 135.89 0)
 		(unit 1)
 		(exclude_from_sim no)
@@
 		(fields_autoplaced yes)
 		(property "Reference" "H4"
-			(at 360.68 139.6999 0)
+			(at 360.68 134.6199 0)
 			(effects
 				(font
@@
 		)
 		(property "Value" "M2.5"
-			(at 360.68 142.2399 0)
+			(at 360.68 137.1599 0)
 			(effects
 				(font
@@
 		)
 		(property "Footprint" "Mounting_Holes:M2.5_Mounting_Hole_2.9mm_unplated"
-			(at 359.156 146.05 0)
+			(at 359.156 140.97 0)
 			(effects
 				(font
@@
 		)
 		(property "Datasheet" ""
-			(at 358.14 140.97 0)
+			(at 358.14 135.89 0)
 			(effects
 				(font
@@
 		)
 		(property "Description" "Mounting Hole M2.5 unplated 2.9mm diameter"
-			(at 358.394 148.336 0)
+			(at 358.394 143.256 0)
 			(effects
 				(font
@@
 	(symbol
 		(lib_id "Mounting_Holes:Mounting_Hole_M2.5")
-		(at 345.44 140.97 0)
+		(at 345.44 135.89 0)
 		(unit 1)
 		(exclude_from_sim no)
@@
 		(fields_autoplaced yes)
 		(property "Reference" "H3"
-			(at 347.98 139.6999 0)
+			(at 347.98 134.6199 0)
 			(effects
 				(font
@@
 		)
 		(property "Value" "M2.5"
-			(at 347.98 142.2399 0)
+			(at 347.98 137.1599 0)
 			(effects
 				(font
@@
 		)
 		(property "Footprint" "Mounting_Holes:M2.5_Mounting_Hole_2.9mm_unplated"
-			(at 346.456 146.05 0)
+			(at 346.456 140.97 0)
 			(effects
 				(font
@@
 		)
 		(property "Datasheet" ""
-			(at 345.44 140.97 0)
+			(at 345.44 135.89 0)
 			(effects
 				(font
@@
 		)
 		(property "Description" "Mounting Hole M2.5 unplated 2.9mm diameter"
-			(at 345.694 148.336 0)
+			(at 345.694 143.256 0)
 			(effects
 				(font
@@
 	)
 	(symbol
+		(lib_id "urchin-logo-sym:LOGO")
+		(at 378.46 260.35 0)
+		(unit 1)
+		(exclude_from_sim no)
+		(in_bom yes)
+		(on_board yes)
+		(dnp no)
+		(fields_autoplaced yes)
+		(property "Reference" "#G1"
+			(at 378.46 252.73 0)
+			(effects
+				(font
+					(size 1.27 1.27)
+				)
+				(hide yes)
+			)
+		)
+		(property "Value" "LOGO"
+			(at 378.46 268.224 0)
+			(effects
+				(font
+					(size 1.27 1.27)
+				)
+				(hide yes)
+			)
+		)
+		(property "Footprint" ""
+			(at 378.46 260.35 0)
+			(effects
+				(font
+					(size 1.27 1.27)
+				)
+				(hide yes)
+			)
+		)
+		(property "Datasheet" ""
+			(at 378.46 260.35 0)
+			(effects
+				(font
+					(size 1.27 1.27)
+				)
+				(hide yes)
+			)
+		)
+		(property "Description" ""
+			(at 378.46 260.35 0)
+			(effects
+				(font
+					(size 1.27 1.27)
+				)
+				(hide yes)
+			)
+		)
+		(instances
+			(project ""
+				(path "/71a801ea-23a0-4bb3-891f-1f0b94a910f4"
+					(reference "#G1")
+					(unit 1)
+				)
+			)
+		)
+	)
+	(symbol
 		(lib_id "power:GND")
 		(at 267.97 198.12 90)
@@
 	(symbol
 		(lib_id "Mounting_Holes:Mounting_Hole_M2.5")
-		(at 332.74 140.97 0)
+		(at 332.74 135.89 0)
 		(unit 1)
 		(exclude_from_sim no)
@@
 		(fields_autoplaced yes)
 		(property "Reference" "H2"
-			(at 335.28 139.6999 0)
+			(at 335.28 134.6199 0)
 			(effects
 				(font
@@
 		)
 		(property "Value" "M2.5"
-			(at 335.28 142.2399 0)
+			(at 335.28 137.1599 0)
 			(effects
 				(font
@@
 		)
 		(property "Footprint" "Mounting_Holes:M2.5_Mounting_Hole_2.9mm_unplated"
-			(at 333.756 146.05 0)
+			(at 333.756 140.97 0)
 			(effects
 				(font
@@
 		)
 		(property "Datasheet" ""
-			(at 332.74 140.97 0)
+			(at 332.74 135.89 0)
 			(effects
 				(font
@@
 		)
 		(property "Description" "Mounting Hole M2.5 unplated 2.9mm diameter"
-			(at 332.994 148.336 0)
+			(at 332.994 143.256 0)
 			(effects
 				(font
@@
 					(unit 1)
 				)
+			)
+		)
+	)
+	(symbol
+		(lib_id "urchin-logo-sym:LOGO")
+		(at 327.66 260.35 0)
+		(unit 1)
+		(exclude_from_sim no)
+		(in_bom yes)
+		(on_board yes)
+		(dnp no)
+		(fields_autoplaced yes)
+		(property "Reference" "#G2"
+			(at 327.66 252.73 0)
+			(effects
+				(font
+					(size 1.27 1.27)
+				)
+				(hide yes)
+			)
+		)
+		(property "Value" "LOGO"
+			(at 327.66 268.224 0)
+			(effects
+				(font
+					(size 1.27 1.27)
+				)
+				(hide yes)
+			)
+		)
+		(property "Footprint" ""
+			(at 327.66 260.35 0)
+			(effects
+				(font
+					(size 1.27 1.27)
+				)
+				(hide yes)
+			)
+		)
+		(property "Datasheet" ""
+			(at 327.66 260.35 0)
+			(effects
+				(font
+					(size 1.27 1.27)
+				)
+				(hide yes)
+			)
+		)
+		(property "Description" ""
+			(at 327.66 260.35 0)
+			(effects
+				(font
+					(size 1.27 1.27)
+				)
+				(hide yes)
+			)
+		)
+		(instances
+			(project ""
+				(path "/71a801ea-23a0-4bb3-891f-1f0b94a910f4"
+					(reference "#G2")
+					(unit 1)
+				)
